File: ecad/mcu.kicad_sch (KiCad schematic)
At the start: 31 parts, among them J1 ST_STDC14, J2 GCT 4105, J3 Conn_01x02, SW1 SW_Push, U13 STM32F405RGTx, Y1 12MHz

Commit message: More work on layout
Parts:
- added JP1, JP2, JP3: SolderJumper_2_Bridged, Jumper:SolderJumper-2_P1.3mm_Bridged_RoundedPad1.0x1.5mm, symbol Jumper:SolderJumper_2_Bridged
- added TP1: TestPoint, TestPoint:TestPoint_Pad_D2.0mm, symbol Connector:TestPoint
- added U14: M24C64-RMN6TP, Package_SO:SOIC-8_3.9x4.9mm_P1.27mm, symbol Memory_NVRAM:FM24C64B
Connections:
- net +3.3V: now also TP1.1, U14.8 (VDD)
- net GND: now also JP1.1 (A), JP2.1 (A), JP3.1 (A), U14.4 (VSS)
- net VCP_RX: now reaches J1.13 (VCP_RX)
- net VCP_TX: now reaches J1.14 (VCP_TX)
- new net: JP2.2 (B), U14.2 (A1)
- new net: JP3.2 (B), U14.3 (A2)
- new net: JP1.2 (B), U14.1 (A0)
- new net EEPROM_SCL: U14.6 (SCL)
- new net EEPROM_SDA: U14.5 (SDA)
- new net EEPROM_WP: U14.7 (WP)
